File: Central_Module.kicad_pcb (KiCad board)
At the start: 2 copper layers, 32.5 x 32.5 mm, 50 parts, among them J1 USB_B_Micro, J2 SM13B-GHS-TB_LF__SN_, J3 Conn_01x01, J4 Conn_01x01, J5 Conn_01x01, J6 Conn_01x01, J7 Conn_01x01, J8 Conn_01x01, J9 Conn_01x01, Q1 AO3401A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

Commit message: Pre-Violations DRC Corrections
Parts:
- moved J6 42.2 mm to (164.0, 91.5)
- moved J7 41.7 mm to (163.5, 106.0)
- moved J5 40.8 mm to (164.0, 93.5)
- moved J3 39.5 mm to (163.5, 103.0)
- moved J4 39.5 mm to (163.5, 104.5)
- moved J8 21.0 mm to (188.5, 90.5)
- moved J9 15.1 mm to (190.0, 107.5)
- moved U1 1.46 mm to (184.0, 95.9)
- moved J2 1.23 mm to (176.8, 86.0)
Routing:
- net /SCL: track 22.7 -> 55.6 mm, vias 2 -> 3
- net /SDA: track 23.8 -> 48.5 mm, vias 2 -> 3
- net /DIN: track 0.90 -> 12.3 mm
- net /RST: track 69.1 -> 59.6 mm, vias 1 -> 2
- net /BCLK: track 0.00 -> 5.09 mm, vias 0 -> 1
- net /LRCLK: track 0.95 -> 5.29 mm
- net /D+: track 10.6 -> 8.86 mm
- net /SCK: track 36.2 -> 35.0 mm
- net /Display_CS: track 12.2 -> 11.0 mm
- net /DC: track 11.8 -> 10.6 mm
- net /MOSI: track 40.9 -> 39.7 mm
- net /D-: track 9.31 -> 8.27 mm
- net /RXD: track 14.0 -> 14.9 mm
- net /TXD: track 12.3 -> 13.2 mm
- net /MISO: track 29.9 -> 30.8 mm
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- added copper zone on F.Cu, net +3.3V
- added copper zone on B.Cu, net GND
Other:
- board size 32.5 x 32.5 mm -> 32.4 x 31.8 mm

Commit message: Post DRC Checker
Parts:
- added R3: 10k, Resistor_SMD:R_0402_1005Metric, B.Cu at (178.0, 96.0)
- moved L1 0.53 mm to (162.5, 96.5)
- moved C4 0.50 mm to (177.5, 102.5)
- moved J9 0.50 mm to (189.5, 107.5)
- moved Q1 0.38 mm to (172.0, 112.6)
Routing:
- net GND: track 0.00 -> 151.9 mm, vias 0 -> 22
- net +3.3V: track 3.50 -> 62.3 mm, vias 1 -> 9
- net TBD: track 9.27 -> 38.7 mm, vias 5 -> 7
- net /CS: track 0.00 -> 15.6 mm, vias 0 -> 2
- net /MISO: track 30.8 -> 46.1 mm, vias 2 -> 3
- net /USB5V: track 40.7 -> 49.3 mm, vias 2 -> 4
- net /RST: track 59.6 -> 64.5 mm
- net /DC: track 10.6 -> 11.5 mm
Other:
- board size 32.4 x 31.8 mm -> 33.6 x 32.8 mm
- board text added: "Angelo Duenas"

Commit message: ForReview
Parts:
- added J10: Conn_01x01, Imports:1mm Pad, F.Cu at (169.0, 112.5)
- added R4: 4.7k, Resistor_SMD:R_0402_1005Metric, F.Cu at (167.5, 111.5)
- moved R2 14.6 mm to (170.0, 104.5), turned to 90 degrees
- moved R1 13.1 mm to (171.5, 104.0), turned to 90 degrees
- moved J7 1.00 mm to (163.5, 107.0)
- moved J4 0.50 mm to (163.5, 105.0)
- moved J9 0.50 mm to (190.0, 107.5)
- moved C16 0.46 mm to (174.0, 103.0)
Connections:
- R1 pad 1: +3.3V -> /SCL
- R1 pad 2: /SCL -> Net-(U5-GPIO9)
- R2 pad 1: +3.3V -> /SDA
- R2 pad 2: /SDA -> Net-(U5-GPIO8)
- U5 pad 14: /SDA -> Net-(U5-GPIO8)
- U5 pad 15: /SCL -> Net-(U5-GPIO9)
Routing:
- net +3.3V: track 62.3 -> 72.7 mm
- net Net-(U5-GPIO8): track 0.00 -> 2.10 mm, vias 0 -> 1
- net /DIN: track 12.3 -> 14.0 mm
- net Net-(J10-Pin_1): track 0.00 -> 1.41 mm
- net Net-(U5-GPIO9): track 0.00 -> 1.39 mm, vias 0 -> 1
- net /RST: track 64.5 -> 65.2 mm
- net TBD: track 38.7 -> 38.0 mm, vias 7 -> 6
- net /SDA: track 48.9 -> 48.4 mm, vias 3 -> 4
- net /SCL: track 56.0 -> 55.5 mm, vias 3 -> 4
- net /LRCLK: track 5.29 -> 5.79 mm
- net GND: track 151.9 -> 152.1 mm, vias 22 -> 21
