File: Central_Module.kicad_sch (KiCad schematic)
At the start: 51 parts, among them J1 USB_B_Micro, J2 SM13B-GHS-TB_LF__SN_, J3 Conn_01x01, J4 Conn_01x01, J5 Conn_01x01, J6 Conn_01x01, J7 Conn_01x01, J8 Conn_01x01, J9 Conn_01x01, Q1 AO3401A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

Commit message: ForReview
Parts:
- added J10: Conn_01x01, Imports:1mm Pad, symbol Connector_Generic:Conn_01x01
- added R4: 4.7k, Resistor_SMD:R_0402_1005Metric, symbol Device:R_US
Connections:
- net +3.3V: now also R4.1; no longer R1.1, R2.1
- net SCL: now also R1.1; no longer R1.2, U5.15 (GPIO9)
- net SDA: now also R2.1; no longer R2.2, U5.14 (GPIO8)
- new net: J10.1 (Pin_1), R4.2
- new net: R1.2, U5.15 (GPIO9)
- new net: R2.2, U5.14 (GPIO8)
Other:
- note removed: "Pull-Up Resistors"
- moved on the sheet: R1, R2
